Commit message: safety

File: src/viz/models/URDF_Simulation/model_V6.urdf (robot description, URDF)
Before this commit: robot converted_robot, 101 links, 100 joints
Links:
- removed link world
- removed link world2root_fixed_jointbody
Joints:
- removed joint world2root_fixed
- removed joint world2root_fixed_offset
- joint root2thumb_base_offset: origin xyz=0.0682 0.0663 -0.009 rpy=0.0 0.0 0.0 -> xyz=0 0 0 rpy=0.0 0.0 0.0
- joint thumb_abd: origin xyz=-0.05696 -0.11383 0.0 rpy=0.0 0.0 0.0 -> xyz=-0.05696 -0.011383 0.0 rpy=0.0 0.0 0.0
- joint thumb_abd_offset: origin xyz=0.05696 0.11383 -0.0 rpy=0.0 0.0 0.0 -> xyz=0 0 0 rpy=0.0 0.0 0.0
- joint thumb_abd_virt: origin xyz=-0.05696 -0.11383 0.0 rpy=0.0 0.0 0.0 -> xyz=0.01388722858794558 -0.0472924545530461 -0.0026400640968846715 rpy=0.0 0.0 0.0
- joint thumb_abd_virt_offset: origin xyz=0.05696 0.11383 -0.0 rpy=0.0 0.0 0.0 -> xyz=0 0 0 rpy=0.0 0.0 0.0
- joint thumb_um2mp_offset: origin xyz=0.062947 0.124166 -0.008 rpy=0.0 0.0 0.0 -> xyz=0 0 0 rpy=0.0 0.0 0.0
- joint thumb_um2mp_virt: origin xyz=-0.072947 -0.114166 0.008 rpy=0.0 0.0 0.0 -> xyz=-0.0 -0.0 0.0 rpy=0.0 0.0 0.0
- joint thumb_um2mp_virt_offset: origin xyz=0.072947 0.114166 -0.008 rpy=0.0 0.0 0.0 -> xyz=0.0 0.0 -0.0 rpy=0.0 0.0 0.0

Commit message: updated urdf

File: src/viz/models/URDF_Simulation/model_V6.urdf (robot description, URDF)
Before this commit: robot converted_robot, 99 links, 98 joints
Joints:
- joint thumb_abd: origin xyz=-0.05696 -0.011383 0.0 rpy=0.0 0.0 0.0 -> xyz=0.008088722858794558 -0.0172924545530461 -0.0026400640968846715 rpy=0.0 0.0 0.0
- joint thumb_abd_virt_offset: origin xyz=0 0 0 rpy=0.0 0.0 0.0 -> xyz=0 -0 0 rpy=0.0 0.0 0.0

Commit message: Change root to hand_root

File: src/viz/models/URDF_Simulation/model_V6.urdf (robot description, URDF)
Before this commit: robot converted_robot, 99 links, 98 joints
Links:
- removed link root
- added link hand_root, mass 0.0
Joints:
- joint root2tower_fixed: parent root -> hand_root
- joint thumb_abd: origin xyz=0.008088722858794558 -0.0172924545530461 -0.0026400640968846715 rpy=0.0 0.0 0.0 -> xyz=0.0021088722858794558 -0.0212924545530461 -0.0026400640968846715 rpy=0.0 0.0 0.0
- joint thumb_abd_virt: origin xyz=0.01388722858794558 -0.0472924545530461 -0.0026400640968846715 rpy=0.0 0.0 0.0 -> xyz=0.007088722858794558 -0.0312924545530461 -0.0026400640968846715 rpy=0.0 0.0 0.0
- joint thumb_um2mp: origin xyz=-0.062947 -0.124166 0.008 rpy=0.0 0.0 0.0 -> xyz=-0.01438088722858794558 -0.0212924545530461 -0.0026400640968846715 rpy=0.0 0.0 0.0
